File: 555_Badge/555_Badge.kicad_pcb (KiCad board)
At the start: 2 copper layers, 59.7 x 27.9 mm, 15 parts, among them Q1 2N3904

Commit message: Added text to board layout
Other:
- board text added: "+"
- board text added: "PCB Design by Michael Probst 12/23/2021"
